File: µSSDV/µSSDV.kicad_pcb (KiCad board)
At the start: 2 copper layers, 26.3 x 40 mm, 12 parts, among them J1 Conn_01x02_Pin, U1 ESP32-CAM, U2 atgm336h gps, U3 RFM98W-433S2, U4 TLV61070ADBV

Commit message: Minor PCB updates
Parts:
- ANT1: value GPS Antenna -> GPS Antenne
- ANT2: value LoRa Antenna -> LoRa Antenne
Connections:
- U1 pad P$15: GPS_TX -> GPS_RX
- U1 pad P$7: GPS_RX -> unconnected-(U1-IO2-PadP$7)
- U2 pad 3: GPS_TX -> unconnected-(U2-RXD1-Pad3)
Routing:
- net GPS_RX: track 27.6 -> 12.6 mm
- net GPS_TX: track 12.2 -> 0.00 mm, vias 1 -> 0
- net SCK: track 11.3 -> 9.86 mm
Changed lines of the file:
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@@
 			(outputformat 1)
 			(mirror no)
-			(drillshape 1)
+			(drillshape 0)
 			(scaleselection 1)
-			(outputdirectory "")
+			(outputdirectory "Gerbers/uSSDV V1.0/")
 		)
 	)
@@
 	(net 12 "RX")
 	(net 13 "IO0")
-	(net 14 "GPS_TX")
+	(net 14 "unconnected-(U1-IO2-PadP$7)")
 	(net 15 "MOSI")
 	(net 16 "CS")
@@
 	(net 35 "unconnected-(U3-DIO0-Pad14)")
 	(net 36 "unconnected-(U3-DIO3-Pad11)")
+	(net 37 "unconnected-(U2-RXD1-Pad3)")
 	(footprint "Connector_PinHeader_2.54mm:PinHeader_1x01_P2.54mm_Vertical"
 		(layer "F.Cu")
@@
 		(tags "Through hole pin header THT 1x01 2.54mm single row")
 		(property "Reference" "ANT1"
-			(at 3.75 0 -0)
+			(at 3.75 0 0)
 			(layer "B.SilkS")
 			(effects
@@
 			)
 		)
-		(property "Value" "GPS Antenna"
+		(property "Value" "GPS Antenne"
 			(at 10.75 0 0)
 			(layer "B.SilkS")
@@
 			(layers "F.Cu" "F.Mask" "F.Paste")
 			(roundrect_rratio 0.25)
-			(net 14 "GPS_TX")
+			(net 37 "unconnected-(U2-RXD1-Pad3)")
 			(pinfunction "RXD1")
-			(pintype "input")
+			(pintype "input+no_connect")
 		)
 		(pad "4" smd roundrect
@@
 			(layers "*.Cu" "*.Mask")
 			(remove_unused_layers no)
-			(net 8 "GPS_RX")
+			(net 14 "unconnected-(U1-IO2-PadP$7)")
 			(pinfunction "IO2")
-			(pintype "bidirectional")
+			(pintype "bidirectional+no_connect")
 			(solder_mask_margin 0.102)
 		)
@@
 			(layers "*.Cu" "*.Mask")
 			(remove_unused_layers no)
-			(net 14 "GPS_TX")
+			(net 8 "GPS_RX")
 			(pinfunction "IO16")
 			(pintype "bidirectional")
@@
 			)
 		)
-		(property "Value" "LoRa Antenna"
+		(property "Value" "LoRa Antenne"
 			(at 7.25 0 0)
 			(layer "F.SilkS")
@@
 	)
 	(segment
-		(start 92.75 52.25)
-		(end 92.9 52.1)
+		(start 97.5 49)
+		(end 98 49)
 		(width 0.2)
 		(layer "F.Cu")
@@
 	)
 	(segment
-		(start 92.9 52.1)
-		(end 94.75 52.1)
+		(start 94.75 52.1)
+		(end 95.749714 52.1)
 		(width 0.2)
 		(layer "F.Cu")
 		(net 8)
 	)
-	(via
-		(at 92.75 52.25)
-		(size 0.6)
-		(drill 0.3)
-		(layers "F.Cu" "B.Cu")
-		(net 8)
-	)
-	(segment
-		(start 83.75 66.5)
-		(end 83.4434 66.8066)
-		(width 0.2)
-		(layer "B.Cu")
-		(net 8)
-	)
-	(segment
-		(start 83.4434 67.651921)
-		(end 83.792479 68.001)
-		(width 0.2)
-		(layer "B.Cu")
-		(net 8)
-	)
 	(segment
-		(start 92.75 59.458521)
-		(end 92.75 52.25)
+		(start 96 50.5)
+		(end 97.5 49)
 		(width 0.2)
-		(layer "B.Cu")
+		(layer "F.Cu")
 		(net 8)
 	)
 	(segment
-		(start 81.82 63.2185)
-		(end 83.75 65.1485)
+		(start 96 51.849714)
+		(end 96 50.5)
 		(width 0.2)
-		(layer "B.Cu")
+		(layer "F.Cu")
 		(net 8)
 	)
 	(segment
-		(start 83.75 65.1485)
-		(end 83.75 66.5)
+		(start 95.749714 52.1)
+		(end 96 51.849714)
 		(width 0.2)
-		(layer "B.Cu")
+		(layer "F.Cu")
 		(net 8)
 	)
-	(segment
-		(start 83.4434 66.8066)
-		(end 83.4434 67.651921)
-		(width 0.2)
-		(layer "B.Cu")
+	(via
+		(at 98 49)
+		(size 0.6)
+		(drill 0.3)
+		(layers "F.Cu" "B.Cu")
 		(net 8)
 	)
 	(segment
-		(start 83.792479 68.001)
-		(end 84.207521 68.001)
+		(start 98 49)
+		(end 99.5185 50.5185)
 		(width 0.2)
 		(layer "B.Cu")
@@
 	)
 	(segment
-		(start 84.207521 68.001)
-		(end 92.75 59.458521)
+		(start 99.5185 50.5185)
+		(end 104.68 50.5185)
 		(width 0.2)
 		(layer "B.Cu")
@@
 	)
 	(segment
-		(start 98.73934 48.45)
-		(end 98.3 48.45)
-		(width 0.2)
-		(layer "F.Cu")
-		(net 14)
-	)
-	(segment
-		(start 98.3 48.45)
-		(end 95.75 51)
-		(width 0.2)
-		(layer "F.Cu")
-		(net 14)
-	)
-	(segment
-		(start 95.75 51)
-		(end 94.75 51)
-		(width 0.2)
-		(layer "F.Cu")
-		(net 14)
-	)
-	(via
-		(at 98.73934 48.45)
-		(size 0.6)
-		(drill 0.3)
-		(layers "F.Cu" "B.Cu")
-		(net 14)
-	)
-	(segment
-		(start 100.2685 50.5185)
-		(end 104.68 50.5185)
-		(width 0.2)
-		(layer "B.Cu")
-		(net 14)
-	)
-	(segment
-		(start 98.73934 48.98934)
-		(end 100.2685 50.5185)
-		(width 0.2)
-		(layer "B.Cu")
-		(net 14)
-	)
-	(segment
-		(start 98.73934 48.45)
-		(end 98.73934 48.98934)
-		(width 0.2)
-		(layer "B.Cu")
-		(net 14)
-	)
-	(segment
 		(start 83.75 66)
 		(end 84.25 66.5)
@@
 	)
 	(segment
-		(start 85.725 65.775)
-		(end 85.725 64.5835)
-		(width 0.2)
-		(layer "B.Cu")
-		(net 18)
-	)
-	(segment
-		(start 85.725 64.5835)
+		(start 84 62.8585)
 		(end 81.82 60.6785)
 		(width 0.2)
@@
 	(segment
 		(start 84 67.5)
-		(end 85.725 65.775)
+		(end 84 62.8585)
 		(width 0.2)
 		(layer "B.Cu")
